File: hardware/can-adapter/adapter1.sch (EAGLE design)
At the start: 7 parts, among them J1 PJ-30220, J2 PJ-30220, J3 PJ-30220

Commit message: chore: fill schematic title blocks with CBA credit and doc numbers
Co-Authored-By: Claude Opus 4.6 <noreply@anthropic.com>
Other:
- note added: "1.0"
- note added: "CAN Bus Academy (canbusacademy.com)"
- note added: "CBA-CAN-ADP-001"
- note added: "Design: Igor Ramos | License: Open Source Hardware"
Changed lines of the file:
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@@
 <sheet>
 <plain>
+<text x="187.96" y="11.43" size="2.54" layer="94" font="vector">CBA-CAN-ADP-001</text>
+<text x="244.475" y="11.43" size="2.54" layer="94" font="vector">1.0</text>
+<text x="148.59" y="30.48" size="2.54" layer="94" font="vector">CAN Bus Academy (canbusacademy.com)</text>
+<text x="148.59" y="25.4" size="1.778" layer="94" font="vector">Design: Igor Ramos | License: Open Source Hardware</text>
 </plain>
 <instances>
