File: hardware/can-adapter/db9_trs_adapter.sch (EAGLE design)
At the start: 7 parts, among them J1 PJ-30220, J2 PJ-30220, J3 PJ-30220

Commit message: docs: explain RING1 vs RING2 rationale, update termination to 120 ohm
- Spec: added section explaining why CAN_L must be on RING1 (RING2
  shorts to GND when TRS plug is inserted into TRRS jack)
- Adapter: default termination changed from 60 to 120 ohm (standard
  CAN endpoint termination), with note on 60 ohm for single-point use

Co-Authored-By: Claude Opus 4.6 <noreply@anthropic.com>
Parts:
- R1: value 60 -> 120
Changed lines of the file:
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@@
 </part>
 <part name="X1" library="SparkFun" deviceset="DB9" device="FEMALE"/>
-<part name="R1" library="rcl" deviceset="R-US_" device="M0805" value="60"/>
+<part name="R1" library="rcl" deviceset="R-US_" device="M0805" value="120"/>
 <part name="RT" library="SparkFun" deviceset="M02" device="PTH"/>
 <part name="J3" library="igor_lib_6d4d0" deviceset="AUDIO_JACK_4POS" device="A" value="PJ-30220">
